File: hardware/elektrosluch.sch (EAGLE design)
At the start: 28 parts, among them IC1 OPA2134UA, X1 STEREOJACK, X2 STEREOJACK

Commit message: Layout tests
Parts:
- removed ALPS_POT: RK0971221Z05, audio-pots:ALPS_RK0971221Z0N
- removed C3, C4: 220uF, rcl:CPOL-EUD
- removed H1, H2, H3, H4: MOUNT-PAD-ROUND3.0, holes:MOUNT-PAD-ROUND3.0
- removed JP1: (no value), pinhead:PINHD-1X2
- removed LED1: LED, mojakniznica:LED
- removed R10, R9: 100k, rcl:R-EU_R0805
- removed R11: 1k, rcl:R-EU_R0805
- removed X1, X2: STEREOJACK, adafruit:STEREOJACK
- added C12, C9: 220uf, SparkFun-Passives:CAP_POLPTH2
- added C15, C16: 100n, TomW:C-EU0805_CAP
- added D1, D2: (no value), diode:DIODE-SOD123
- added F1, F2: PTCSMD, SparkFun-PowerIC:PTCSMD
- added POWER: (no value), TomW:10_PIN_HEADER
- added RV1: (no value), SparkFun-Electromechanical:POT_DUAL
- added U$1, U$6, U$7: THONKICONNNEW, MusicThingModular:THONKICONNNEW
- U$2: value BATT -> THONKICONNNEW; device mojakniznica:BATT -> MusicThingModular:THONKICONNNEW
Connections:
- removed net +5V: ALPS_POTG$3.S1, C3.+, IC1A.V+, R11.2, R9.2
- removed net -5V: C4.-, IC1A.V-, JP1.1, LED1.C, R10.1
- new net +12V: C15.2, C9.+, D2.C, F1.1, IC1A.V+
- new net -12V: C12.-, C16.1, D1.A, F2.1, IC1A.V-
- net GND: now also C12.+, C15.1, C16.2, C9.-, D1.C, D2.A, POWER.3, POWER.4, POWER.5, POWER.6, POWER.7, POWER.8, RV1G$1.A, RV1G$2.A, U$1.TIP, U$2.TIP, U$6.SLEEVE, U$7.SLEEVE; no longer ALPS_POTL.1, ALPS_POTR.1, C3.-, C4.+, H1.MOUNT, H2.MOUNT, H3.MOUNT, H4.MOUNT, R10.2, R9.1, X1.1, X2.1
- net N$10: now also U$2.SWITCH; no longer X1.2
- net N$12: now also U$1.SWITCH; no longer X1.4
- net N$13: now also U$2.SLEEVE; no longer X1.3
- net N$14: now also F1.2, POWER.10, POWER.9; no longer LED1.A, R11.1
- net N$16: now also F2.2, POWER.1, POWER.2; no longer ALPS_POTG$3.S2, JP1.2
- net N$3: now also RV1G$1.E; no longer ALPS_POTL.3
- net N$6: now also RV1G$2.E; no longer ALPS_POTR.3
- net N$7: now also RV1G$1.S, U$6.TIP; no longer ALPS_POTL.2, X2.5
- net N$8: now also U$1.SLEEVE; no longer X1.5
- net N$9: now also RV1G$2.S, U$7.TIP; no longer ALPS_POTR.2, X2.2
Other:
- note removed: "9V battery"
